Commit message: camera added to urdf

File: hoverboard_demo_description/urdf/ros2_control/ros2_control.urdf.xacro (robot description, xacro)
@@ -5,18 +5,18 @@
       <hardware>
         <plugin>hoverboard_hardware_interface/HoverboardHardwareInterface</plugin>
-        <param name="left_wheel_joint_name">driving_wheel_left_joint</param>
-        <param name="right_wheel_joint_name">driving_wheel_right_joint</param>
+        <param name="left_wheel_joint_name">left_wheel_joint</param>
+        <param name="right_wheel_joint_name">right_wheel_joint</param>
         <param name="loop_rate">50</param>
-        <param name="device">/dev/ttyUSB0</param>
+        <param name="device">/dev/ttyUSB-myftdi</param>
         <param name="baud_rate">115200</param>
         <param name="timeout">1000</param>
         <param name="encoder_ticks_per_revolution">90</param>
       </hardware>
-      <joint name="driving_wheel_left_joint">
+      <joint name="left_wheel_joint">
         <command_interface name="velocity"/>
         <state_interface name="position"/>
         <state_interface name="velocity"/>
       </joint>
-      <joint name="driving_wheel_right_joint">
+      <joint name="right_wheel_joint">
         <command_interface name="velocity"/>
         <state_interface name="position"/>
